File: hardware/3x2/audio_controller_3x2.kicad_pcb (KiCad board)
At the start: 2 copper layers, 69.8 x 40.6 mm, 15 parts, among them P1 HEADER_02X08_SMD, SW1 SPST_SLIDE_AS, U1 TLE7230R

Commit message: teensy -> 3x2.
Parts:
- C1, C2: footprint audio_controller_teensy:SM1210 -> audio_controller_3x2:SM1210
- L1, L2, L3, L4, L5, L6, L7, L8, L9: footprint audio_controller_teensy:LED_555-3XXX -> audio_controller_3x2:LED_555-3XXX
- MDT1: footprint audio_controller_teensy:MODULAR_DEVICE_TEENSY_MALE -> audio_controller_3x2:MODULAR_DEVICE_TEENSY_MALE
- P1: footprint audio_controller_teensy:HEADER_02x08_SMD -> audio_controller_3x2:HEADER_02x08_SMD
- SW1: footprint audio_controller_teensy:SPST_SLIDE_AS -> audio_controller_3x2:SPST_SLIDE_AS
- U1: footprint audio_controller_teensy:PG-DSO-36 -> audio_controller_3x2:PG-DSO-36
Other:
- board text added: "Janelia Modular Device audio_controller model_number: 1111 08/2016 ver 1.1 3x2"
- board text removed: "Janelia Modular Device audio_controller model_number: 1111 08/2016 ver 1.1 teensy"
Changed lines of the file:
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@@
   (page A4)
   (title_block
-    (title audio_controller_teensy)
+    (title audio_controller_3x2)
     (rev 1.1)
   )
@@
     (add_net VDD)
   )
-  (module audio_controller_teensy:SM1210 (layer B.Cu)
+  (module audio_controller_3x2:SM1210 (layer B.Cu)
     (at 85.725 91.44 180)
     (tags "CMS SM")
@@
     )
   )
-  (module audio_controller_teensy:SM1210 (layer B.Cu)
+  (module audio_controller_3x2:SM1210 (layer B.Cu)
     (at 128.905 107.95)
     (tags "CMS SM")
@@
     )
   )
-  (module audio_controller_teensy:LED_555-3XXX (layer F.Cu)
+  (module audio_controller_3x2:LED_555-3XXX (layer F.Cu)
     (at 84.455 99.695 180)
     (fp_text reference L1 (at 0 -5.08 90) (layer F.SilkS)
@@
       (net 1 GND))
   )
-  (module audio_controller_teensy:LED_555-3XXX (layer F.Cu)
+  (module audio_controller_3x2:LED_555-3XXX (layer F.Cu)
     (at 117.475 106.045 180)
     (fp_text reference L2 (at -2.54 0 90) (layer F.SilkS)
@@
       (net 5 /OUT0))
   )
-  (module audio_controller_teensy:LED_555-3XXX (layer F.Cu)
+  (module audio_controller_3x2:LED_555-3XXX (layer F.Cu)
     (at 114.935 106.045 180)
     (fp_text reference L3 (at 0 -5.842 270) (layer F.SilkS) hide
@@
       (net 6 /OUT1))
   )
-  (module audio_controller_teensy:LED_555-3XXX (layer F.Cu)
+  (module audio_controller_3x2:LED_555-3XXX (layer F.Cu)
     (at 112.395 106.045 180)
     (fp_text reference L4 (at 0 -5.842 270) (layer F.SilkS) hide
@@
       (net 7 /OUT2))
   )
-  (module audio_controller_teensy:LED_555-3XXX (layer F.Cu)
+  (module audio_controller_3x2:LED_555-3XXX (layer F.Cu)
     (at 109.855 106.045 180)
     (fp_text reference L5 (at 0 -5.842 270) (layer F.SilkS) hide
@@
       (net 8 /OUT3))
   )
-  (module audio_controller_teensy:LED_555-3XXX (layer F.Cu)
+  (module audio_controller_3x2:LED_555-3XXX (layer F.Cu)
     (at 107.315 106.045 180)
     (fp_text reference L6 (at 0 -5.842 270) (layer F.SilkS) hide
@@
       (net 9 /OUT4))
   )
-  (module audio_controller_teensy:LED_555-3XXX (layer F.Cu)
+  (module audio_controller_3x2:LED_555-3XXX (layer F.Cu)
     (at 104.775 106.045 180)
     (fp_text reference L7 (at 0 -5.842 270) (layer F.SilkS) hide
@@
       (net 10 /OUT5))
   )
-  (module audio_controller_teensy:LED_555-3XXX (layer F.Cu)
+  (module audio_controller_3x2:LED_555-3XXX (layer F.Cu)
     (at 102.235 106.045 180)
     (fp_text reference L8 (at 0 -5.842 270) (layer F.SilkS) hide
@@
       (net 11 /OUT6))
   )
-  (module audio_controller_teensy:LED_555-3XXX (layer F.Cu)
+  (module audio_controller_3x2:LED_555-3XXX (layer F.Cu)
     (at 99.695 106.045 180)
     (fp_text reference L9 (at 2.54 0 90) (layer F.SilkS)
@@
       (net 12 /OUT7))
   )
-  (module audio_controller_teensy:HEADER_02x08_SMD (layer F.Cu)
+  (module audio_controller_3x2:HEADER_02x08_SMD (layer F.Cu)
     (at 108.585 96.52)
     (fp_text reference P1 (at 15.24 3.81 90) (layer F.SilkS)
@@
       (net 12 /OUT7))
   )
-  (module audio_controller_teensy:SPST_SLIDE_AS (layer F.Cu)
+  (module audio_controller_3x2:SPST_SLIDE_AS (layer F.Cu)
     (at 88.265 99.695)
     (fp_text reference SW1 (at 3.81 0 90) (layer F.SilkS)
@@
       (net 4 /LED_PWR))
   )
-  (module audio_controller_teensy:PG-DSO-36 (layer B.Cu)
+  (module audio_controller_3x2:PG-DSO-36 (layer B.Cu)
     (at 128.905 96.52 270)
     (fp_text reference U1 (at -6.75 -6.75 180) (layer B.SilkS)
@@
       (net 1 GND) (solder_mask_margin 0.05) (clearance 0.05))
   )
-  (module audio_controller_teensy:MODULAR_DEVICE_TEENSY_MALE (layer F.Cu)
+  (module audio_controller_3x2:MODULAR_DEVICE_TEENSY_MALE (layer F.Cu)
     (at 95.25 99.695)
     (fp_text reference MDT1 (at 0 0) (layer F.SilkS) hide
@@
     (effects (font (thickness 0.381)) (justify left))
   )
-  (gr_text "Janelia Modular Device\naudio_controller\nmodel_number: 1111\n08/2016 ver 1.1 teensy" (at 77.47 99.695 90) (layer F.SilkS)
+  (gr_text "Janelia Modular Device\naudio_controller\nmodel_number: 1111\n08/2016 ver 1.1 3x2" (at 77.47 99.695 90) (layer F.SilkS)
     (effects (font (size 1.016 1.016) (thickness 0.254)))
   )
